File: schematic/Chessfield/Chessfield.kicad_sch (KiCad schematic)
At the start: 13 parts, among them J1 Conn_01x04_Pin, J2 Conn_01x04_Pin, J3 Conn_01x04_Pin, J4 Conn_01x04_Pin

Commit message: update chesssfield
Connections:
- net DIS is gone; now on net DIL: J3.3 (Pin_3)
Changed lines of the file:
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@@
 		)
 	)
-	(global_label "DIS"
+	(global_label "DIL"
 		(shape input)
 		(at 124.46 127 270)
@@
 		)
 		(property "Intersheetrefs" "${INTERSHEET_REFS}"
-			(at 124.46 133.0695 90)
+			(at 124.46 132.8881 90)
 			(effects
 				(font

Commit message: finish chessfield
Parts:
- H1: footprint Package_TO_SOT_THT:TO-92_Inline -> Package_TO_SOT_THT:TO-92_Inline_Horizontal1
Other:
- moved on the sheet: C1, C2, C3, C4, D1, D2, D3, D4, H1, J1, J2, J3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
